File: brainfreeze.kicad_pcb (KiCad board)
At the start: 4 copper layers, 50 x 90 mm, 26 parts, among them J1 Conn_01x01_Pin, J10 Conn_01x01_Pin, J11 Conn_01x01_Pin, J12 Conn_01x01_Pin, J13 Conn_01x01_Pin, J2 Conn_01x01_Pin, J3 Conn_01x01_Pin, J4 Conn_01x01_Pin, J5 Conn_01x01_Pin, J6 Conn_01x01_Socket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

Commit message: Updated PCB
Parts:
- removed J12, J13: Conn_01x01_Pin, Connector_Wire:SolderWire-0.5sqmm_1x01_D0.9mm_OD2.1mm
- removed J9: Conn_01x01_Socket, Connector_Wire:SolderWire-1sqmm_1x01_D1.4mm_OD2.7mm
- A1: footprint Module:Arduino_Nano -> brainfreeze:NANO_FIT
- J6: value Conn_01x01_Socket -> Conn_01x03_Socket; footprint Connector_Wire:SolderWire-1sqmm_1x01_D1.4mm_OD2.7mm -> brainfreeze:ESC CON
- J7: value Conn_01x01_Pin -> Conn_01x03_Socket; footprint Connector_Wire:SolderWire-0.5sqmm_1x01_D0.9mm_OD2.1mm -> brainfreeze:ESC CON
- moved A1 28.9 mm to (201.3, 142.0)
- moved J6 22.0 mm to (177.0, 81.5), turned to 90 degrees
- moved J7 0.72 mm to (177.1, 92.6), turned to 90 degrees
Connections:
- net SOLDERPAD renamed NEOPIXEL LED
- A1 pad 11: unconnected-(A1-D8-Pad11) -> ESC_2
- A1 pad 12: unconnected-(A1-D9-Pad12) -> ESC_1
- A1 pad 14: unconnected-(A1-D11-Pad14) -> LED
- A1 pad 9: LED -> unconnected-(A1-D6-Pad9)
- J6 pad 1: +12V -> +5V
- J7 pad 1: ESC_SIGNAL1 -> +5V
Routing:
- net ESC_SIGNAL2: track 93.3 -> 0.00 mm, vias 1 -> 0
- net ESC_SIGNAL3: track 67.4 -> 0.00 mm, vias 1 -> 0
- net ESC_1: track 0.00 -> 64.9 mm
- net ESC_2: track 0.00 -> 51.2 mm, vias 0 -> 1
- net ESC_SIGNAL1: track 41.9 -> 0.00 mm
- net LED: track 14.2 -> 26.6 mm, vias 2 -> 1
- net +5V: track 29.0 -> 36.0 mm, vias 2 -> 4
Other:
- board text added: "3V3"
- board text added: "ESC_1"
- board text added: "ESC_2"
- board text added: "GND"
- board text added: "HI-PWR LED SCREW CON"
- board text added: "INT1"
- board text added: "PWR"
- board text added: "PWR INDICATOR LED"
- board text added: "SCL"
- board text added: "SDA"
- board text added: "SIG"
- board text added: "STATUS LED"
- board text removed: "ESC POWER"
- board text removed: "ESC SIGNAL1"
- board text removed: "ESC SIGNAL2"
- board text removed: "ESC SIGNAL3"
- board text removed: "LED CONNECTOR"
- board text removed: "NEOPIXEL"
- board text removed: "RESISTOR AND LED"
