File: brainfreeze/brainfreeze.kicad_sch (KiCad schematic)
At the start: 13 parts, among them J1 XT30PW-M, P1 OSTTE020104, Q1 DMN63D8L-7, U1 H3LIS331DL, U3 AP63205WU

Commit message: Created gerber files
Parts:
- removed J1: XT30PW-M, brainfreeze:XT30PW-M, symbol XT30PW-M:XT30PW-M
- added J1, J10, J11, J3, J4, J5: Conn_01x01_Pin, Connector_Wire:SolderWire-1sqmm_1x01_D1.4mm_OD2.7mm, symbol Connector:Conn_01x01_Pin
- added J2, J8: Conn_01x01_Pin, Connector_Wire:SolderWire-0.5sqmm_1x01_D0.9mm_OD2.1mm, symbol Connector:Conn_01x01_Pin
- added J6, J7: Conn_01x03_Socket, brainfreeze:ESC CON, symbol Connector:Conn_01x03_Socket
- A1: footprint Module:Arduino_Nano -> brainfreeze:NANO_FIT
Connections:
- net +12V: now also J1.1 (Pin_1)
- net +5V: now also J10.1 (Pin_1), J3.1 (Pin_1), J6.1 (Pin_1), J7.1 (Pin_1)
- net GND: now also J11.1 (Pin_1), J4.1 (Pin_1), J5.1 (Pin_1), J6.3 (Pin_3), J7.3 (Pin_3)
- net LED: now also A1.14 (D11); no longer A1.9 (D6)
- net ESC_2: now reaches A1.11 (D8)
- net ESC_2: now also J7.2 (Pin_2)
- net ESC_1: now reaches A1.12 (D9)
- net ESC_1: now also J6.2 (Pin_2)
- net NEOPIXEL LED: now reaches A1.16 (D13)
- net NEOPIXEL LED: now also J2.1 (Pin_1)
- net RX: now reaches A1.2 (D0/RX)
- net RX: now also J8.1 (Pin_1)
- net ESC_SIGNAL1: now reaches A1.5 (D2)
- no-connect marks 24 -> 19
Other:
- note added: "ESC CONNECTORS"
- note added: "PWR INDICATOR LED"
- note added: "RECIEVER"
- note added: "Solder Pads for NeoPixel LED"
- note added: "https://www.flysky-cn.com/fsi6x"
- note removed: "Indicator LED"
- moved on the sheet: C1, C2, C3, C4, L1, Q1, U1, U3
